File: pcb/angelina_integrated.kicad_pcb (KiCad board)
At the start: 2 copper layers, 381.9 x 126.1 mm, 147 parts, among them J1 MJ-4PP-9, P1 i2c-pin-A, P2 i2c-pin-B, SW1 SW_PUSH, SW10 SW_PUSH, SW11 SW_PUSH, SW12 SW_PUSH, SW13 SW_PUSH, SW14 SW_PUSH, SW15 SW_PUSH, SW16 SW_PUSH, SW17 SW_PUSH, SW18 SW_PUSH, SW19 SW_PUSH, SW2 SW_PUSH, SW20 SW_PUSH, SW21 SW_PUSH, SW22 SW_PUSH, SW23 SW_PUSH, SW24 SW_PUSH, SW25 SW_PUSH, SW26 SW_PUSH, SW27 SW_PUSH, SW28 SW_PUSH, SW29 SW_PUSH, SW3 SW_PUSH, SW30 SW_PUSH, SW31 SW_PUSH, SW32 SW_PUSH, SW33 SW_PUSH, SW34 SW_PUSH, SW35 SW_PUSH, SW36 SW_PUSH, SW37 SW_PUSH, SW38 SW_PUSH, SW39 SW_PUSH, SW4 SW_PUSH, SW40 SW_PUSH, SW41 SW_PUSH, SW42 SW_PUSH, SW43 SW_PUSH, SW44 SW_PUSH, SW45 SW_PUSH, SW46 SW_PUSH, SW47 SW_PUSH, SW48 SW_PUSH, SW49 SW_PUSH, SW5 SW_PUSH, SW50 SW_PUSH, SW51 SW_PUSH, SW52 SW_PUSH, SW53 SW_PUSH, SW54 SW_PUSH, SW55 SW_PUSH, SW56 SW_PUSH, SW57 SW_PUSH, SW58 SW_PUSH, SW59 SW_PUSH, SW6 SW_PUSH, SW60 SW_PUSH, SW61 SW_PUSH, SW62 SW_PUSH, SW63 SW_PUSH, SW64 SW_PUSH, SW65 SW_PUSH, SW66 SW_PUSH, SW67 SW_PUSH, SW68 SW_PUSH, SW7 SW_PUSH, SW8 SW_PUSH, SW9 SW_PUSH, U1 ProMicro_r

Commit message: Fix pcb
Parts:
- moved P1 4.21 mm to (229.8, 77.7)
- moved R1 4.21 mm to (235.4, 77.7)
- moved JP1 2.74 mm to (219.4, 77.6)
- moved P2 1.07 mm to (229.8, 75.0)
- moved R2 1.07 mm to (235.4, 75.0)
- moved RSW1 0.89 mm to (195.9, 77.4)
Routing:
- net VCC: track 48.0 -> 42.0 mm
- net SCL: track 24.6 -> 28.7 mm
- net Net-(J1-PadA): track 11.0 -> 7.07 mm
- net SDA: track 25.4 -> 22.8 mm
- net data: track 5.66 -> 3.09 mm
- net reset: track 5.76 -> 4.87 mm

Commit message: Finished to make pcb
Parts:
- moved JP1 11.8 mm to (208.4, 81.9), turned to 180 degrees
- moved RSW1 5.27 mm to (192.3, 73.5), turned to 180 degrees
- moved J1 1.49 mm to (223.2, 71.7)
- moved P1 1.19 mm to (228.6, 77.7)
- moved P2 1.19 mm to (228.6, 75.0)
- moved R1 1.19 mm to (234.3, 77.7)
- moved R2 1.19 mm to (234.3, 75.0)
Routing:
- net reset: track 4.87 -> 29.2 mm
- net VCC: track 42.0 -> 25.2 mm
- net col0: track 294.3 -> 278.7 mm
- net Net-(J1-PadB): track 11.8 -> 26.6 mm
- net SDA: track 22.8 -> 36.6 mm
- net SCL: track 28.7 -> 42.1 mm
- net data: track 3.09 -> 8.57 mm
Other:
- outline, holes or cut-outs redrawn

Commit message: Add credit
Parts:
- added REF**: credit, angelina_integerated:credit, F.Cu at (164.9, 73.5)
Changed lines of the file:
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@@
   (general
     (thickness 1.6)
-    (drawings 0)
+    (drawings 2)
     (tracks 558)
     (zones 0)
-    (modules 147)
+    (modules 148)
     (nets 90)
   )
@@
     (visible_elements FFFFFFFF)
     (pcbplotparams
-      (layerselection 0x010fc_ffffffff)
+      (layerselection 0x010f0_ffffffff)
       (usegerberextensions false)
       (usegerberattributes false)
@@
       (outputformat 1)
       (mirror false)
-      (drillshape 1)
+      (drillshape 0)
       (scaleselection 1)
-      (outputdirectory ""))
+      (outputdirectory "../output/"))
   )
   (net 0 "")
@@
     (add_net VCC)
   )
+  (module angelina_integerated:credit (layer F.Cu)
+    (at 164.901424 73.521032)
+    (fp_text reference REF** (at 0 1.016) (layer F.Fab) hide
+      (effects (font (size 1 1) (thickness 0.15)))
+    )
+    (fp_text value credit (at 0 -1.016) (layer F.Fab) hide
+      (effects (font (size 1 1) (thickness 0.15)))
+    )
+    (fp_text user "Angelina Integrated rev.1 (2020.06) Designed by clomie" (at 0 0) (layer B.Mask)
+      (effects (font (size 1 1) (thickness 0.15)) (justify mirror))
+    )
+  )
   (module angelina_integerated:ProMicro (layer F.Cu)
     (at 208.3592 71.735096)
@@
       (net 80 col2))
   )
+  (dimension 96.142904 (width 0.15) (layer F.Fab)
+    (gr_text "96.143 mm" (at 16.55936 119.806548 270) (layer F.Fab)
+      (effects (font (size 1 1) (thickness 0.15)))
+    )
+    (feature1 (pts (xy 22.3242 167.878) (xy 17.272939 167.878)))
+    (feature2 (pts (xy 22.3242 71.735096) (xy 17.272939 71.735096)))
+    (crossbar (pts (xy 17.85936 71.735096) (xy 17.85936 167.878)))
+    (arrow1a (pts (xy 17.85936 167.878) (xy 17.272939 166.751496)))
+    (arrow1b (pts (xy 17.85936 167.878) (xy 18.445781 166.751496)))
+    (arrow2a (pts (xy 17.85936 71.735096) (xy 17.272939 72.8616)))
+    (arrow2b (pts (xy 17.85936 71.735096) (xy 18.445781 72.8616)))
+  )
+  (dimension 381.893024 (width 0.15) (layer F.Fab)
+    (gr_text "381.893 mm" (at 212.079712 64.18432) (layer F.Fab)
+      (effects (font (size 1 1) (thickness 0.15)))
+    )
+    (feature1 (pts (xy 403.026224 72.9257) (xy 403.026224 64.897899)))
+    (feature2 (pts (xy 21.1332 72.9257) (xy 21.1332 64.897899)))
+    (crossbar (pts (xy 21.1332 65.48432) (xy 403.026224 65.48432)))
+    (arrow1a (pts (xy 403.026224 65.48432) (xy 401.89972 66.070741)))
+    (arrow1b (pts (xy 403.026224 65.48432) (xy 401.89972 64.897899)))
+    (arrow2a (pts (xy 21.1332 65.48432) (xy 22.259704 66.070741)))
+    (arrow2b (pts (xy 21.1332 65.48432) (xy 22.259704 64.897899)))
+  )
   (segment (start 48.815584 84.54524) (end 48.815584 77.092904) (width 0.25) (layer B.Cu) (net 1))
